Commit message: feature: mycobot320_description funcional pkg with the display.launch.py to see the robot and test it with sliders in rviz

File: src/mycobot320_ros2/mycobot320_description/urdf/mech/mycobot320_arm.urdf.xacro (robot description, xacro)
@@ -1,134 +1,142 @@
-<xml version="1.0"?>
+<?xml version="1.0"?>
 <robot xmlns:xacro="http://www.ros.org/wiki/xacro" name="mycobot320">
-    <link name="link1">
-        <visual>
-            <geometry>
-                <mesh filename="package://mycobot320_description/meshes/mycobot320/visual/link1.dae"/>
-            </geometry>
-            <origin xyz = "0.0 0.0 -0.078 " rpy = " 0 0 1.5708"/>
-        </visual>
-        <collision>
-            <origin xyz = "0.0 0.0 -0.078 " rpy = " 0 0 1.5708"/>
-            <geometry>
-                <!--<mesh    filename="package://mycobot320_description/meshes/mycobot320/visual/link1.dae"/>-->
-                <cylinder length="0.106" radius="0.043"/>
-            </geometry>
-        </collision>
-    </link>
-    <link name="link2">
-        <visual>
-            <geometry>
-                <mesh filename="package://mycobot320_description/meshes/mycobot320/visual/link2.dae"/>
-            </geometry>
-            <origin xyz = "0.0 0.0 -0.04 " rpy = " 0 1.5708 0"/>
-        </visual>
-        <collision>
-            <origin xyz = "0.0 0.0 -0.04 " rpy = " 0 1.5708 d0"/>
-            <geometry>
-                <!--<mesh    filename="package://mycobot320_description/meshes/mycobot320/visual/link2.dae"/>-->
-                <cylinder length="0.18" radius="0.036"/>
-            </geometry>
-        </collision>
-    </link>
-    <link name="link3">
-        <visual>
-            <geometry>
-                <mesh filename="package://mycobot320_description/meshes/mycobot320/visual/link3.dae"/>
-            </geometry>
-            <origin xyz = "0.0 0.0 0.039 " rpy = " 1.5708 1.5708 1.5708"/>
-        </visual>
-        <collision>
-            <geometry>
-                <!--<mesh    filename="package://mycobot320_description/meshes/mycobot320/visual/link3.dae"/>-->
-                <cylinder length="0.14" radius="0.0305"/>
-            </geometry>
-            <origin xyz = "0.0 0.0 0.039 " rpy = " 1.5708 1.5708 1.5708"/>
-        </collision>
-    </link>
-    <link name="link4">
-        <visual>
-            <geometry>
-                <mesh filename="package://mycobot320_description/meshes/mycobot320/visual/link4.dae"/>
-            </geometry>
-            <origin xyz = "0.0 -0.0024 -0.05" rpy = " 1.5708 1.5708 0"/>
-        </visual>
-        <collision>
-            <geometry>
-                <!--<mesh    filename="package://mycobot320_description/meshes/mycobot320/visual/link4.dae"/>-->
-                <cylinder length="0.083" radius="0.029"/>
-            </geometry>
-            <origin xyz = "0.0 -0.0024 -0.05" rpy = " 1.5708 1.5708 0"/>
-        </collision>
-    </link>
-    <link name="link5">
-        <visual>
-            <geometry>
-                <mesh filename="package://mycobot320_description/meshes/mycobot320/visual/link5.dae"/>
-            </geometry>
-            <origin xyz = "0.0 0.0 -0.05 " rpy = " 0    0 -1.5708"/>
-        </visual>
-        <collision>
-            <geometry>
-                <cylinder length="0.0849" radius="0.029"/>
-                <!--<mesh    filename="package://mycobot320_description/meshes/mycobot320/visual/link5.dae"/>-->
-            </geometry>
-            <origin xyz = "0.0 0.0 -0.05 " rpy = " 0    0 -1.5708"/>
-        </collision>
-    </link>
-    <link name="link6">
-        <visual>
-            <geometry>
-                <mesh filename="package://mycobot320_description/meshes/mycobot320/visual/link6.dae"/>
-            </geometry>
-         <origin xyz = "0.0 0.0 -0.0115 " rpy = " 1.5708 1.5708 0"/>
-        </visual>
-        <collision>
-            <geometry>
-                <cylinder length="0.0225" radius="0.026"/>
-                <!--<mesh    filename="package://mycobot320_description/meshes/mycobot320/visual/link6.dae"/>-->
-            </geometry>
-            <origin xyz = "0.0 0.0 -0.0115 " rpy = " 1.5708 1.5708 0"/>
-        </collision>
-    </link>
-    <joint name="joint2_to_joint1" type="revolute">
-        <axis xyz="0 0 1"/>
-        <limit effort = "1000.0" lower = "-2.9321" upper = "2.9321" velocity = "0"/>
-        <parent link="base"/>
-        <child link="link1"/>
-        <origin xyz= "0 0 0.173" rpy = "0 0 0"/>
-    </joint>
-    <joint name="joint3_to_joint2" type="revolute">
-        <axis xyz="0 0 1"/>
-        <limit effort = "1000.0" lower = "-2.3561" upper = "2.3561" velocity = "0"/>
-        <parent link="link1"/>
-        <child link="link2"/>
-        <origin xyz= "0 -0.086 0" rpy = "0 -1.5708 1.5708"/>
-    </joint>
-    <joint name="joint4_to_joint3" type="revolute">
-        <axis xyz=" 0 0 1"/>
-        <limit effort = "1000.0" lower = "-2.5307" upper = "2.5307" velocity = "0"/>
-        <parent link="link2"/>
-        <child link="link3"/>
-        <origin xyz= "0.13635 0 -0.086     " rpy = "0 0 0"/>
-    </joint>
-    <joint name="joint5_to_joint4" type="revolute">
-        <axis xyz=" 0 0 1"/>
-        <limit effort = "1000.0" lower = "-2.5830" upper = "2.5830" velocity = "0"/>
-        <parent link="link3"/>
-        <child link="link4"/>
-        <origin xyz = "0.1195 0 0.082 " rpy = " 0 0 1.57080"/>
-    </joint>
-    <joint name="joint6_to_joint5" type="revolute">
-        <axis xyz="0 0 1"/>
-        <limit effort = "1000.0" lower = "-2.9321" upper = "2.9321" velocity = "0"/>
-        <parent link="link4"/>
-        <child link="link5"/>
-        <origin xyz= "0 -0.09415 0.0" rpy = "1.5708 0 0"/>
-    </joint>
-    <joint name="joint6output_to_joint6" type="revolute">
-        <axis xyz="0 0 1"/>
-        <limit effort = "1000.0" lower = "-3.14159" upper = "3.14159" velocity = "0"/>
-        <parent link="link5"/>
-        <child link="link6"/>
-        <origin xyz= "0 0.055 0.0" rpy = "-1.5708 0 0"/>
-    </joint>
+    <xacro:macro name="cylinder_link" params="name mesh origin rpy collision_origin collision_rpy length radius ">
+        <link name="${name}">
+            <visual>
+                <geometry>
+                    <mesh filename="${mesh}"/>
+                </geometry>
+                <origin xyz="${origin}" rpy="${rpy}"/>
+            </visual>
+            <collision>
+                <origin xyz="${collision_origin}"  rpy="${collision_rpy}"/>
+                <geometry>
+                    <!--<mesh filename="${mesh}"/>-->
+                    <cylinder length="${length}" radius="${radius}"/>
+                </geometry>
+            </collision>
+        </link>
+    </xacro:macro>
+    <!--
+    original_length = 0.09
+    length = original_length + 3/4 radius
+    collision_origin = {0,0,-original_length/2+radius/2}-->
+    <xacro:cylinder_link
+        name="link1"
+        mesh="package://mycobot320_description/meshes/mycobot320/visual/link1.dae"
+        origin="0.0 0.0 -0.078"
+        rpy="0 0 1.5708"
+        collision_origin="0.0 0.0 -0.0235"
+        collision_rpy="0 0 1.5708"
+        length="0.12375"
+        radius="0.04"/>
+    <!--All length, radius and collion pose had been graphically obtained.-->
+    <xacro:cylinder_link
+        name="link2"
+        mesh="package://mycobot320_description/meshes/mycobot320/visual/link2.dae"
+        origin="0.0 0.0 -0.04"
+        rpy="0 1.5708 0"
+        collision_origin="0.065 0.0 0.0005"
+        collision_rpy="0 1.5708 0"
+        length="0.2"
+        radius="0.0315"/>
+    <xacro:cylinder_link
+        name="link3"
+        mesh="package://mycobot320_description/meshes/mycobot320/visual/link3.dae"
+        origin="0.0 0.0 0.039"
+        rpy="1.5708 1.5708 1.5708"
+        collision_origin="0.06 0.0 -0.005"
+        collision_rpy="1.5708 1.5708 1.5708"
+        length="0.175"
+        radius="0.03"/>
+    <xacro:cylinder_link
+        name="link4"
+        mesh="package://mycobot320_description/meshes/mycobot320/visual/link4.dae"
+        origin="0.0 -0.0024 -0.05"
+        rpy="1.5708 1.5708 0"
+        collision_origin="0.0 -0.0234 -0.0"
+        collision_rpy="1.5708 1.5708 0"
+        length="0.095"
+        radius="0.029"/>
+    <xacro:cylinder_link
+        name="link5"
+        mesh="package://mycobot320_description/meshes/mycobot320/visual/link5.dae"
+        origin="0.0 0.0 -0.05"
+        rpy="0 0 -1.5708"
+        collision_origin="0.0 -0.008 0"
+        collision_rpy="0 1.5708 -1.5708"
+        length="0.08"
+        radius="0.029"/>
+    <xacro:cylinder_link
+        name="link6"
+        mesh="package://mycobot320_description/meshes/mycobot320/visual/link6.dae"
+        origin="0.0 0.0 -0.022"
+        rpy="1.5708 1.5708 0"
+        collision_origin="0.0 0.0 -0.0125"
+        collision_rpy="0 0 0"
+        length="0.015"
+        radius="0.03"/>
+    <xacro:macro name="revolute_joint" params="name parent child origin rpy axis lower upper">
+        <joint name="${name}" type="revolute">
+            <parent link="${parent}"/>
+            <child link="${child}"/>
+            <origin xyz="${origin}" rpy="${rpy}"/>
+            <axis xyz="${axis}"/>
+            <limit lower="${lower}" upper="${upper}" effort="999.0" velocity="0"/>
+        </joint>
+    </xacro:macro>
+    <xacro:revolute_joint
+        name="joint1"
+        parent="base"
+        child="link1"
+        origin="0 0 0.173"
+        rpy="0 0 0"
+        axis="0 0 1"
+        lower="-2.9321"
+        upper="2.9321"/>
+    <xacro:revolute_joint
+        name="joint2"
+        parent="link1"
+        child="link2"
+        origin="0 -0.086 0"
+        rpy="0 -1.5708 1.5708"
+        axis="0 0 1"
+        lower="-2.3561"
+        upper="2.3561"/>
+    <xacro:revolute_joint
+        name="joint3"
+        parent="link2"
+        child="link3"
+        origin="0.13635 0 -0.086"
+        rpy="0 0 0"
+        axis="0 0 1"
+        lower="-2.5307"
+        upper="2.5307"/>
+    <xacro:revolute_joint
+        name="joint4"
+        parent="link3"
+        child="link4"
+        origin="0.1195 0 0.082"
+        rpy="0 0 1.57080"
+        axis="0 0 1"
+        lower="-2.5830"
+        upper="2.5830"/>
+    <xacro:revolute_joint
+        name="joint5"
+        parent="link4"
+        child="link5"
+        origin="0 -0.09415 0.0"
+        rpy="1.5708 0 0"
+        axis="0 0 1"
+        lower="-2.9321"
+        upper="2.9321"/>
+    <xacro:revolute_joint
+        name="joint6"
+        parent="link5"
+        child="link6"
+        origin="0 0.055 0.0"
+        rpy="-1.5708 0 0"
+        axis="0 0 1"
+        lower="-3.14159"
+        upper="3.14159"/>
+</robot>

File: src/mycobot320_ros2/mycobot320_description/urdf/mech/mycobot320_base.urdf.xacro (robot description, xacro)
@@ -10,8 +10,8 @@
     <collision>
       <geometry>
-        <cylinder length="0.102" radius="0.0725"/>
+        <cylinder length="0.09" radius="0.0725"/>
         <!--<mesh filename="package://mycobot320_description/meshes/mycobot320/visual/base.dae"/>-->
       </geometry>
-      <origin xyz="0.0 0 0" rpy="0 0 1.5708"/>
+      <origin xyz="0.0 0 0.045" rpy="0 0 1.5708"/>
     </collision>
   </link>

File: src/mycobot320_ros2/mycobot320_description/urdf/robots/mycobot320.urdf.xacro (robot description, xacro)
@@ -1,6 +1,13 @@
 <?xml version="1.0"?>
 <robot xmlns:xacro="http://www.ros.org/wiki/xacro" name="mycobot320">
-  <xacro:include filename="../mech/mycobot320_base.urdf.xacro"/>
-  <xacro:include filename="../mech/mycobot320_arm.urdf.xacro"/>
-  <xacro:include filename="../mech/mycobot320_gripper.urdf.xacro"/>
+    <xacro:include filename="$(find mycobot320_description)/urdf/mech/mycobot320_base.urdf.xacro"/>
+    <xacro:include filename="$(find mycobot320_description)/urdf/mech/mycobot320_arm.urdf.xacro"/>
+    <!--<xacro:include filename="$(find mycobot320_description)/urdf/mech/mycobot320_gripper.urdf.xacro"/>-->
+    <!-- Define the base link for moveit, gazebo, ros2_control, etc...-->
+    <link name="base_link"/>
+    <joint name="base_link_to_base" type="fixed">
+        <parent link="base_link"/>
+        <child link="base"/>
+        <origin xyz="0 0 0" rpy="0 0 0"/>
+    </joint>
 </robot>

Commit message: improvement: change 1.5708 radians to ${pi/2}

File: src/mycobot320_ros2/mycobot320_description/urdf/mech/mycobot320_arm.urdf.xacro (robot description, xacro)
@@ -26,7 +26,7 @@
         mesh="package://mycobot320_description/meshes/mycobot320/visual/link1.dae"
         origin="0.0 0.0 -0.078"
-        rpy="0 0 1.5708"
+        rpy="0 0 ${pi/2}"
         collision_origin="0.0 0.0 -0.0235"
-        collision_rpy="0 0 1.5708"
+        collision_rpy="0 0 ${pi/2}"
         length="0.12375"
         radius="0.04"/>
@@ -36,7 +36,7 @@
         mesh="package://mycobot320_description/meshes/mycobot320/visual/link2.dae"
         origin="0.0 0.0 -0.04"
-        rpy="0 1.5708 0"
+        rpy="0 ${pi/2} 0"
         collision_origin="0.065 0.0 0.0005"
-        collision_rpy="0 1.5708 0"
+        collision_rpy="0 ${pi/2} 0"
         length="0.2"
         radius="0.0315"/>
@@ -45,7 +45,7 @@
         mesh="package://mycobot320_description/meshes/mycobot320/visual/link3.dae"
         origin="0.0 0.0 0.039"
-        rpy="1.5708 1.5708 1.5708"
+        rpy="${pi/2} ${pi/2} ${pi/2}"
         collision_origin="0.06 0.0 -0.005"
-        collision_rpy="1.5708 1.5708 1.5708"
+        collision_rpy="${pi/2} ${pi/2} ${pi/2}"
         length="0.175"
         radius="0.03"/>
@@ -54,7 +54,7 @@
         mesh="package://mycobot320_description/meshes/mycobot320/visual/link4.dae"
         origin="0.0 -0.0024 -0.05"
-        rpy="1.5708 1.5708 0"
+        rpy="${pi/2} ${pi/2} 0"
         collision_origin="0.0 -0.0234 -0.0"
-        collision_rpy="1.5708 1.5708 0"
+        collision_rpy="${pi/2} ${pi/2} 0"
         length="0.095"
         radius="0.029"/>
@@ -63,7 +63,7 @@
         mesh="package://mycobot320_description/meshes/mycobot320/visual/link5.dae"
         origin="0.0 0.0 -0.05"
-        rpy="0 0 -1.5708"
+        rpy="0 0 -${pi/2}"
         collision_origin="0.0 -0.008 0"
-        collision_rpy="0 1.5708 -1.5708"
+        collision_rpy="0 ${pi/2} -${pi/2}"
         length="0.08"
         radius="0.029"/>
@@ -72,5 +72,5 @@
         mesh="package://mycobot320_description/meshes/mycobot320/visual/link6.dae"
         origin="0.0 0.0 -0.022"
-        rpy="1.5708 1.5708 0"
+        rpy="${pi/2} ${pi/2} 0"
         collision_origin="0.0 0.0 -0.0125"
         collision_rpy="0 0 0"
@@ -100,5 +100,5 @@
         child="link2"
         origin="0 -0.086 0"
-        rpy="0 -1.5708 1.5708"
+        rpy="0 -${pi/2} ${pi/2}"
         axis="0 0 1"
         lower="-2.3561"
@@ -118,5 +118,5 @@
         child="link4"
         origin="0.1195 0 0.082"
-        rpy="0 0 1.57080"
+        rpy="0 0 ${pi/2}0"
         axis="0 0 1"
         lower="-2.5830"
@@ -127,5 +127,5 @@
         child="link5"
         origin="0 -0.09415 0.0"
-        rpy="1.5708 0 0"
+        rpy="${pi/2} 0 0"
         axis="0 0 1"
         lower="-2.9321"
@@ -136,5 +136,5 @@
         child="link6"
         origin="0 0.055 0.0"
-        rpy="-1.5708 0 0"
+        rpy="-${pi/2} 0 0"
         axis="0 0 1"
         lower="-3.14159"

File: src/mycobot320_ros2/mycobot320_description/urdf/mech/mycobot320_base.urdf.xacro (robot description, xacro)
@@ -6,5 +6,5 @@
         <mesh filename="package://mycobot320_description/meshes/mycobot320/visual/base.dae"/>
       </geometry>
-      <origin xyz="0.0 0 0" rpy="0 0 1.5708"/>
+      <origin xyz="0.0 0 0" rpy="0 0 ${pi/2}"/>
     </visual>
     <collision>
@@ -13,5 +13,5 @@
         <!--<mesh filename="package://mycobot320_description/meshes/mycobot320/visual/base.dae"/>-->
       </geometry>
-      <origin xyz="0.0 0 0.045" rpy="0 0 1.5708"/>
+      <origin xyz="0.0 0 0.045" rpy="0 0 ${pi/2}"/>
     </collision>
   </link>

File: src/mycobot320_ros2/mycobot320_description/urdf/mech/mycobot320_gripper.urdf.xacro (robot description, xacro)
@@ -7,5 +7,5 @@
                 <mesh filename="package://mycobot320_description/meshes/mycobot320/visual/gripper_base.dae"/>
             </geometry>
-            <origin xyz = "-0.02 0.012 -0.018 " rpy = " 0 0 1.5708"/>
+            <origin xyz = "-0.02 0.012 -0.018 " rpy = " 0 0 ${pi/2}"/>
         </visual>
         <collision>
@@ -14,5 +14,5 @@
                 <mesh filename="package://mycobot320_description/meshes/mycobot320/visual/gripper_base.dae"/>
             </geometry>
-            <origin xyz = "-0.02 0.012 -0.018 " rpy = " 0 0 1.5708"/>
+            <origin xyz = "-0.02 0.012 -0.018 " rpy = " 0 0 ${pi/2}"/>
         </collision>
     </link>
@@ -23,5 +23,5 @@
                 <mesh filename="package://mycobot320_description/meshes/mycobot320/visual/gripper_left1.dae"/>
             </geometry>
-            <origin xyz = "0.036 -0.052 0.0 " rpy = " 0 0 1.5708"/>
+            <origin xyz = "0.036 -0.052 0.0 " rpy = " 0 0 ${pi/2}"/>
         </visual>
         <collision>
@@ -29,5 +29,5 @@
                 <mesh filename="package://mycobot320_description/meshes/mycobot320/visual/gripper_left1.dae"/>
             </geometry>
-            <origin xyz = "0.036 -0.052 0.0 " rpy = " 0 0 1.5708"/>
+            <origin xyz = "0.036 -0.052 0.0 " rpy = " 0 0 ${pi/2}"/>
         </collision>
     </link>
@@ -37,5 +37,5 @@
                 <mesh filename="package://mycobot320_description/meshes/mycobot320/visual/gripper_left2.dae"/>
             </geometry>
-            <origin xyz = "0.03 0.024 -0.018 " rpy = " 0 0 1.5708"/>
+            <origin xyz = "0.03 0.024 -0.018 " rpy = " 0 0 ${pi/2}"/>
         </visual>
         <collision>
@@ -43,5 +43,5 @@
                 <mesh filename="package://mycobot320_description/meshes/mycobot320/visual/gripper_left2.dae"/>
             </geometry>
-            <origin xyz = "0.03 0.024 -0.018 " rpy = " 0 0 1.5708"/>
+            <origin xyz = "0.03 0.024 -0.018 " rpy = " 0 0 ${pi/2}"/>
         </collision>
     </link>
@@ -51,5 +51,5 @@
                 <mesh filename="package://mycobot320_description/meshes/mycobot320/visual/gripper_left3.dae"/>
             </geometry>
-            <origin xyz = "0.034 0.0 -0.012 " rpy = " 0 3.14159 -1.5708"/>
+            <origin xyz = "0.034 0.0 -0.012 " rpy = " 0 3.14159 -${pi/2}"/>
             <!-- <origin xyz = "0.0 0 0 " rpy = " 0 0 0"/> -->
         </visual>
@@ -58,5 +58,5 @@
                 <mesh filename="package://mycobot320_description/meshes/mycobot320/visual/gripper_left3.dae"/>
             </geometry>
-            <origin xyz = "0.034 0.0 -0.012 " rpy = " 0 3.14159 -1.5708"/>
+            <origin xyz = "0.034 0.0 -0.012 " rpy = " 0 3.14159 -${pi/2}"/>
         </collision>
     </link>
@@ -67,5 +67,5 @@
                 <mesh filename="package://mycobot320_description/meshes/mycobot320/visual/gripper_right1.dae"/>
             </geometry>
-            <origin xyz = "-0.072 -0.05 0.0 " rpy = " 0 0 1.5708"/>
+            <origin xyz = "-0.072 -0.05 0.0 " rpy = " 0 0 ${pi/2}"/>
         </visual>
         <collision>
@@ -73,5 +73,5 @@
                 <mesh filename="package://mycobot320_description/meshes/mycobot320/visual/gripper_right1.dae"/>
             </geometry>
-            <origin xyz = "-0.072 -0.05 0.0 " rpy = " 0 0 1.5708"/>
+            <origin xyz = "-0.072 -0.05 0.0 " rpy = " 0 0 ${pi/2}"/>
         </collision>
     </link>
@@ -81,5 +81,5 @@
                 <mesh filename="package://mycobot320_description/meshes/mycobot320/visual/gripper_right2.dae"/>
             </geometry>
-            <origin xyz = "-0.066 0.023 -0.018 " rpy = " 0 0 1.5708"/>
+            <origin xyz = "-0.066 0.023 -0.018 " rpy = " 0 0 ${pi/2}"/>
         </visual>
         <collision>
@@ -87,5 +87,5 @@
                 <mesh filename="package://mycobot320_description/meshes/mycobot320/visual/gripper_right2.dae"/>
             </geometry>
-            <origin xyz = "-0.066 0.023 -0.018 " rpy = " 0 0 1.5708"/>
+            <origin xyz = "-0.066 0.023 -0.018 " rpy = " 0 0 ${pi/2}"/>
         </collision>
     </link>
@@ -95,5 +95,5 @@
                 <mesh filename="package://mycobot320_description/meshes/mycobot320/visual/gripper_right3.dae"/>
             </geometry>
-            <origin xyz = "0 0.0 -0.012 " rpy = " 0 3.14159 -1.5708"/>
+            <origin xyz = "0 0.0 -0.012 " rpy = " 0 3.14159 -${pi/2}"/>
         </visual>
         <collision>
@@ -101,5 +101,5 @@
                 <mesh filename="package://mycobot320_description/meshes/mycobot320/visual/gripper_right3.dae"/>
             </geometry>
-        <origin xyz = "0.0 0.0 -0.012 " rpy = " 0 3.14159 -1.5708"/>
+        <origin xyz = "0.0 0.0 -0.012 " rpy = " 0 3.14159 -${pi/2}"/>
         </collision>
     </link>
@@ -109,5 +109,5 @@
         <parent link="link6"/>
         <child link="gripper_base"/>
-        <origin xyz= "0 0.0 0.042" rpy = "1.5708 0 0"/>
+        <origin xyz= "0 0.0 0.042" rpy = "${pi/2} 0 0"/>
     </joint>
     <joint name="gripper_controller" type="revolute">

Commit message: debug: change q's limit to +- pi for easy debugging without limitations

File: src/mycobot320_ros2/mycobot320_description/urdf/mech/mycobot320_arm.urdf.xacro (robot description, xacro)
@@ -83,5 +83,6 @@
             <origin xyz="${origin}" rpy="${rpy}"/>
             <axis xyz="${axis}"/>
-            <limit lower="${lower}" upper="${upper}" effort="999.0" velocity="0"/>
+            <!--<limit lower="${lower}" upper="${upper}" effort="999.0" velocity="0"/>-->
+            <limit lower="-${pi}" upper="${pi}" effort="999.0" velocity="0"/>
         </joint>
     </xacro:macro>
